Commit message: Update Gazebo world and URDF for refined object and robot configuration

File: src/sortibot_arm/urdf/sortibot_4dof.urdf (robot description, URDF)
Before this commit: robot sortibot_arm, 8 links, 7 joints
Links:
- link camera_link: mass None -> 0.01
- link gripper_body: mass None -> 0.1
Joints:
- joint joint4: axis (none) -> 0 1 0; limit (none) -> lower=-1.57 upper=1.57 effort=5 velocity=1.0; type fixed -> revolute
